Commit message: Complete

File: install/acr_core/share/acr_core/urdf/acr_rrbot.urdf (robot description, URDF)
Before this commit: robot acr_rrbot, 5 links, 4 joints
Links:
- added link lidar_link; visual box size=0.12 0.10 0.07
Joints:
- added joint lidar_fixed: type fixed, parent tool0, child lidar_link, origin xyz=0.10 0 0.14 rpy=0 0 0
